File: pcb/ir-remote.kicad_pcb (KiCad board)
At the start: 2 copper layers, 114.5 x 39.6 mm, 91 parts, among them J12 Conn_01x04, J3 Conn_02x04, J4 USB-C_Receptacle_Molex_217179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, U1 STM32G431CBTx, U112 TLV61046ADB, U2 TSOP38238, U3 NE5532, U4 NE5532, U6 USBLC6-2SC6, U7 DRV8210DRLR, U9 PCM3060PW, X10 16MHz_18pF_FA238

Commit message: PCB WIP
Parts:
- removed C100, C102, C41, C42, C45: 100nF_0402_16V, 4ms_Capacitor:C_0402
- removed C104, C105, C125, C126: 1uF_0402_25V, 4ms_Capacitor:C_0402
- removed C115, C116: 1.5nF_0402_50V, 4ms_Capacitor:C_0402
- removed C121, C122, C123, C124: 560pF_0402_50v, 4ms_Capacitor:C_0402
- removed C44: 22uF_0805_25V, 4ms_Capacitor:C_0805
- removed C49: 2.2uF_0603_25V, 4ms_Capacitor:C_0603
- removed C51: 10uF_0603_10V, 4ms_Capacitor:C_0603
- removed D101, D102: BAT54S, 4ms_Package_SOT:SOT23-3_PO132
- removed NT1: NetTie_2, NetTie:NetTie-2_SMD_Pad0.5mm
- removed R105, R109, R110, R112, R113, R114, R124, R125: 100k_0402, 4ms_Resistor:R_0402
- removed R115, R126: 1k_0402, 4ms_Resistor:R_0402
- removed R119, R120, R121, R122: 10k_0603, 4ms_Resistor:R_0603
- removed R128, R131, R132, R135: 7.5k_0402, 4ms_Resistor:R_0402
- removed R129, R130, R133, R134: 820Ω_0402, 4ms_Resistor:R_0402
- removed R139, R140: 100Ω_0603, 4ms_Resistor:R_0603
- removed R141, R142: 47k_0603, 4ms_Resistor:R_0603
- removed R47, R48: 4.7k_0402, 4ms_Resistor:R_0402
- removed U9: PCM3060PW, Package_SO:TSSOP-28_4.4x9.7mm_P0.65mm
- removed V1: AP2120N-5.0TRG1, 4ms_Package_SOT:SOT23-3_PO132
- added C10: 10uF_0603_10V, 4ms_Capacitor:C_0603, F.Cu at (146.3, 75.9)
- added C11: 10uF_0603_10V, 4ms_Capacitor:C_0603, F.Cu at (140.4, 70.2)
- added C12: 0.1uF_0603_16V, 4ms_Capacitor:C_0603, F.Cu at (145.9, 71.5)
- added C13: 10uF_0603_10V, 4ms_Capacitor:C_0603, F.Cu at (144.2, 80.1)
- added C14: 0.1uF_0603_16V, 4ms_Capacitor:C_0603, F.Cu at (151.8, 69.1)
- added C15: 10uF_0603_10V, 4ms_Capacitor:C_0603, F.Cu at (149.4, 71.5)
- added C16: 1uF_0603_25V, 4ms_Capacitor:C_0603, F.Cu at (147.6, 71.5)
- added C17: 22uF_1206_25V, 4ms_Capacitor:C_1206, F.Cu at (135.6, 91.2)
- added C18: 22uF_1206_25V, 4ms_Capacitor:C_1206, F.Cu at (139.9, 91.2)
- added C19: 1uF_0603_25V, 4ms_Capacitor:C_0603, F.Cu at (120.3, 80.6)
- added C20: 1uF_0603_25V, 4ms_Capacitor:C_0603, F.Cu at (131.7, 80.1)
- added C21: 1uF_0603_25V, 4ms_Capacitor:C_0603, F.Cu at (168.0, 82.2)
- added C22: 47nF_0603_35V, 4ms_Capacitor:C_0603, F.Cu at (170.8, 86.0)
- added C23: 47nF_0603_35V, 4ms_Capacitor:C_0603, F.Cu at (155.8, 86.2)
- added C26: 1uF_0603_25V, 4ms_Capacitor:C_0603, F.Cu at (153.9, 82.3)
- added C27: 10uF_0603_10V, 4ms_Capacitor:C_0603, F.Cu at (172.3, 72.0)
- added C28: 10uF_0603_10V, 4ms_Capacitor:C_0603, F.Cu at (178.0, 71.0)
- added C29: 10uF_0603_10V, 4ms_Capacitor:C_0603, F.Cu at (168.9, 70.8)
- added C30: 10uF_0603_10V, 4ms_Capacitor:C_0603, F.Cu at (163.0, 71.8)
- added C32: 1uF_0603_25V, 4ms_Capacitor:C_0603, F.Cu at (153.8, 71.6)
- added C33: 0.1uF_0603_16V, 4ms_Capacitor:C_0603, F.Cu at (121.8, 56.9)
- added C7: 47pF_0603_50V, 4ms_Capacitor:C_0603, F.Cu at (135.6, 75.3)
- added C8: 47pF_0603_50V, 4ms_Capacitor:C_0603, F.Cu at (135.6, 76.9)
- added C9: 0.1uF_0603_16V, 4ms_Capacitor:C_0603, F.Cu at (139.5, 80.2)
- added J1: Conn_01x02, 4ms_Connector:Pins_1x02_2.54mm_TH, F.Cu at (158.9, 73.3)
- added J2: Conn_01x02, 4ms_Connector:Pins_1x02_2.54mm_TH, F.Cu at (159.0, 76.5)
- added J5: Jack_RCA_Stereo, 4ms_Jack:RCA_Stereo_SwitchCraft-PJRAS2X1S, B.Cu at (118.3, 91.4)
- added J6: Conn_01x03, 4ms_Connector:Pins_1x03_2.54mm_TH, F.Cu at (137.6, 95.0)
- added J7: Jack_RCA_Stereo, 4ms_Jack:RCA_Stereo_SwitchCraft-PJRAS2X1S, B.Cu at (163.9, 91.4)
- added J8: Conn_01x02, 4ms_Connector:Pins_1x02_2.54mm_TH, F.Cu at (97.9, 87.6)
- added JP1: SolderJumper_2_Open, 4ms_SolderJumper:JUMPER_SMD_1x2, F.Cu at (143.4, 67.1)
- added NT2: NetTie, 4ms_SolderJumper:NetTie-2_SMD_Pad0.16mm_6mil, F.Cu at (151.6, 73.1)
- added R10: 1k_0603, 4ms_Resistor:R_0603, F.Cu at (119.4, 77.7)
- added R11: 1k_0603, 4ms_Resistor:R_0603, F.Cu at (130.5, 77.2)
- added R12: 4.7k_0603, 4ms_Resistor:R_0603, F.Cu at (139.0, 67.3)
- added R13: 100Ω_0603, 4ms_Resistor:R_0603, F.Cu at (170.7, 82.2)
- added R14: 100k_0603, 4ms_Resistor:R_0603, F.Cu at (118.1, 80.7)
- added R15: 100k_0603, 4ms_Resistor:R_0603, F.Cu at (129.5, 80.0)
- added R16: 100Ω_0603, 4ms_Resistor:R_0603, F.Cu at (157.1, 82.4)
- added R2: 27Ω_0603, 4ms_Resistor:R_0603, F.Cu at (127.1, 65.3)
- added R3: 27Ω_0603, 4ms_Resistor:R_0603, F.Cu at (125.5, 65.3)
- added R6: 27Ω_0603, 4ms_Resistor:R_0603, F.Cu at (132.0, 65.3)
- added R7: 27Ω_0603, 4ms_Resistor:R_0603, F.Cu at (130.4, 65.3)
- added R8: 27Ω_0603, 4ms_Resistor:R_0603, F.Cu at (128.7, 65.4)
- added R9: 4.7k_0603, 4ms_Resistor:R_0603, F.Cu at (140.9, 67.2)
- added TP1: TestPoint, 4ms_TestPoint:TestPoint_WireHole, F.Cu at (165.0, 81.0)
- added TP11: TestPoint, 4ms_TestPoint:TestPoint_WireHole, F.Cu at (146.9, 88.4)
- added TP12: TestPoint, 4ms_TestPoint:TestPoint_WireHole, F.Cu at (147.0, 84.9)
- added TP13: TestPoint, 4ms_TestPoint:TestPoint_WireHole, F.Cu at (143.7, 85.0)
- added TP14: TestPoint, 4ms_TestPoint:TestPoint_WireHole, F.Cu at (143.7, 91.8)
- added TP2: TestPoint, 4ms_TestPoint:TestPoint_WireHole, F.Cu at (150.9, 81.5)
- added TP3: TestPoint, 4ms_TestPoint:TestPoint_WireHole, F.Cu at (120.2, 74.5)
- added TP4: TestPoint, 4ms_TestPoint:TestPoint_WireHole, F.Cu at (130.5, 73.7)
- added TP5: TestPoint, 4ms_TestPoint:TestPoint_WireHole, F.Cu at (143.8, 94.8)
- added TP6: TestPoint, 4ms_TestPoint:TestPoint_WireHole, F.Cu at (146.5, 94.8)
- added TP7: TestPoint, 4ms_TestPoint:TestPoint_WireHole, F.Cu at (146.7, 91.8)
- added TP8: TestPoint, 4ms_TestPoint:TestPoint_WireHole, F.Cu at (143.9, 88.5)
- added U5: TLV320AIC3204, Package_DFN_QFN:QFN-32-1EP_5x5mm_P0.5mm_EP3.45x3.45mm_ThermalVias, F.Cu at (141.4, 75.3)
- added U8: TAR5S33U, 4ms_Package_SOT:SOT-563-5, F.Cu at (151.4, 71.5)
- U3, U4: value NE5532 -> TLV74018; footprint Package_SO:SOIC-8_5.3x5.3mm_P1.27mm -> 4ms_Package_SOT:SOT-23-5
- moved C2 149.2 mm to (175.1, 48.2), turned to 180 degrees
- moved U3 141.7 mm to (175.1, 72.1), turned to 180 degrees
- moved U4 139.4 mm to (166.0, 71.8), turned to 180 degrees
- moved C3 91.8 mm to (118.3, 66.7), turned to 180 degrees
- moved C1 83.3 mm to (109.5, 63.7), turned to 90 degrees
- moved J4 82.5 mm to (89.9, 93.7)
- moved U6 82.4 mm to (90.0, 86.4)
- moved R1 61.4 mm to (94.5, 87.1), turned to 90 degrees
- moved J3 36.9 mm to (102.1, 46.9), turned to 90 degrees
- moved C38 25.8 mm to (143.6, 48.9)
- moved C39 23.8 mm to (141.4, 49.4)
- moved V11 23.6 mm to (146.9, 52.1)
- moved C35 23.6 mm to (150.2, 49.8)
- moved C36 23.6 mm to (143.4, 54.2)
- moved L11 23.6 mm to (146.9, 47.6)
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Connections:
- C303 pad 1: VDD -> /Vmotor
- C6 pad 1: VDD -> /Vmotor
- POT1 pad T: (no net) -> unconnected-(POT1D-Touch-PadT)
- R4 pad 1: VDD -> /Vmotor
- U1 pad 45: unconnected-(U1-PB8-Pad45) -> /CODEC_RESET
- U112 pad 5: VDD -> /Vmotor
- U3 pad 1: Net-(U3A--) -> /V_USB
- U3 pad 2: Net-(U3A--) -> GND
- U3 pad 3: Net-(D102-AK) -> /V_USB
- U3 pad 4: GND -> unconnected-(U3-NC-Pad4)
- U3 pad 5: Net-(D101-AK) -> /AVDD
- U4 pad 1: Net-(C123-Pad1) -> /V_USB
- U4 pad 2: Net-(U4A--) -> GND
- U4 pad 3: Net-(U4A-+) -> /V_USB
- U4 pad 4: GND -> unconnected-(U4-NC-Pad4)
- U4 pad 5: Net-(U4B-+) -> /DVDD
- U7 pad 5: VDD -> /Vmotor
Routing:
- net /Vmotor: track 0.00 -> 6.43 mm
- net VDD: track 6.43 -> 0.00 mm
Other:
- board size 114.5 x 39.6 mm -> 114.5 x 54.3 mm

Commit message: PCB WIP
Parts:
- moved J3 24.3 mm to (107.4, 70.6), turned to -90 degrees
- moved J12 17.8 mm to (120.2, 69.9)
- moved TP5 1.86 mm to (144.2, 93.0)
- moved TP6 1.81 mm to (146.7, 93.0)
- moved TP14 1.42 mm to (144.2, 90.5)
- moved TP7 1.40 mm to (146.7, 90.5)
- moved C17 0.96 mm to (134.7, 91.3)
- moved C13 0.94 mm to (145.1, 79.8), turned to 0 degrees
- moved C3 0.94 mm to (119.2, 67.0)
- moved C33 0.91 mm to (122.7, 56.8)
- moved TP8 0.63 mm to (144.2, 87.9)
- moved TP13 0.58 mm to (144.2, 85.4)
- moved C18 0.55 mm to (139.4, 91.4)
- moved TP12 0.54 mm to (146.7, 85.4)
- moved TP11 0.48 mm to (146.7, 87.9)
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Connections:
- C40 pad 1: VDD -> /V_USB
- V12 pad 1: VDD -> /V_USB
Routing:
- net /LINEOUT_R: track 0.00 -> 14.0 mm
- net Net-(C23-Pad1): track 0.00 -> 6.63 mm
- net GNDA: track 0.00 -> 5.23 mm
- net Net-(C26-Pad2): track 0.00 -> 3.82 mm

Commit message: PCB routed and ready for review
Parts:
- added C34: 100nF_0603_16V, 4ms_Capacitor:C_0603, F.Cu at (109.4, 53.8)
- J3: value Conn_02x04 -> Pins_02x04_P2.54mm_SMT; footprint 4ms_Connector:Pins_2x04_2.54mm_TH -> 4ms_Connector:Pins_2x04_P2.54mm_Vertical_SMD
- moved J3 22.2 mm to (101.3, 49.3)
- moved TP13 20.6 mm to (131.5, 69.1)
- moved TP11 19.5 mm to (144.8, 68.5)
- moved TP12 19.1 mm to (136.6, 69.1)
- moved J8 15.4 mm to (82.6, 89.0)
- moved R1 14.4 mm to (80.2, 88.8)
- moved R9 11.3 mm to (149.9, 74.0), turned to 180 degrees
- moved JP1 11.1 mm to (149.9, 76.1), turned to 180 degrees
- moved R3 10.9 mm to (136.4, 66.3), turned to 0 degrees
- moved C29 9.84 mm to (177.3, 75.9)
- moved C30 9.36 mm to (171.1, 76.6)
- moved U4 9.36 mm to (174.0, 76.6)
- moved R2 9.29 mm to (136.4, 64.7), turned to 0 degrees
- moved TP5 8.73 mm to (135.6, 94.4)
- moved TP8 8.73 mm to (135.6, 89.3)
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Connections:
- C21 pad 1: /LINEOUT_L -> /LINEOUT_R
- C26 pad 1: /LINEOUT_R -> /LINEOUT_L
- C27 pad 1: /AVDD -> /DVDD
- C30 pad 1: /DVDD -> /AVDD
- C31 pad 2: ADCGND -> +3V3REF
- J1 pad 2: /DVDD -> /AVDD
- J2 pad 2: /AVDD -> /DVDD
- POT1 pad 1: ADCGND -> +3V3REF
- POT1 pad 3: +3V3REF -> ADCGND
- TP1 pad 1: /LINEOUT_L -> /LINEOUT_R
- TP14 pad 1: /MICBIAS -> /IN2_R
- TP2 pad 1: /LINEOUT_R -> /LINEOUT_L
- TP6 pad 1: /IN2_R -> /IN3_R
- TP8 pad 1: /IN3_R -> /MICBIAS
- U3 pad 5: /AVDD -> /DVDD
- U4 pad 5: /DVDD -> /AVDD
Routing:
- net GND: track 16.0 -> 507.4 mm, vias 3 -> 29
- net /V_USB: track 4.18 -> 265.8 mm, vias 0 -> 11
- net GNDA: track 5.23 -> 167.0 mm, vias 0 -> 6
- net +3V3: track 0.00 -> 158.9 mm, vias 0 -> 10
- net ADCGND: track 0.00 -> 94.8 mm, vias 0 -> 3
- net /IR_DEMOD: track 0.00 -> 76.5 mm, vias 0 -> 1
- net /USB_DM: track 0.00 -> 48.5 mm
- net /USB_DP: track 0.00 -> 47.1 mm
- net +3V3REF: track 0.00 -> 45.4 mm
- net /CODEC_RESET: track 0.00 -> 38.2 mm
- net /Slider_ADC: track 0.00 -> 34.4 mm
- net Net-(U7-OUT2): track 0.00 -> 30.7 mm
- net /I2C_SDA: track 0.00 -> 30.1 mm, vias 0 -> 2
- net /I2C_SCL: track 0.00 -> 28.1 mm, vias 0 -> 2
- net /INL: track 0.00 -> 25.7 mm
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Other:
- board size 114.5 x 54.3 mm -> 127.9 x 54.1 mm
- board text added: "AVDD"
- board text added: "D2"
- board text added: "D3"
- board text added: "DVDD"
- board text added: "GND>"
- board text added: "GPIO"
- board text added: "HEADPHONES"
- board text added: "IN2"
- board text added: "IN3"
- board text added: "L"
- board text added: "LDO-EN"
- board text added: "LiL"
- board text added: "LiR"
- board text added: "LoL"
- board text added: "LoR"
- board text added: "MICBIAS"
- board text added: "MISO"
- board text added: "R"
- board text added: "RX"
- board text added: "SCK"
- board text added: "SWD"
- board text added: "TX"
- board text added: "USB-SHLD-GND"

Commit message: Adjust PCB edges and mounting holes to fit enclosure
Parts:
- added H1: MountingHole, 4ms_Hardware:MountingHole_Screw_3mmHole_5.3mmHead, F.Cu at (64.2, 47.3)
- added H2: MountingHole, 4ms_Hardware:MountingHole_Screw_3mmHole_5.3mmHead, F.Cu at (184.0, 53.0)
- added H3: MountingHole, 4ms_Hardware:MountingHole_Screw_3mmHole_5.3mmHead, F.Cu at (184.0, 92.8)
- added H4: MountingHole, 4ms_Hardware:MountingHole_Screw_3mmHole_5.3mmHead, F.Cu at (64.2, 92.8)
- U2: moved to B.Cu
- moved C22 7.66 mm to (177.2, 81.7)
- moved C23 6.58 mm to (160.7, 81.8), turned to 0 degrees
- moved U2 3.75 mm to (181.3, 46.5), turned to 0 degrees
- moved C2 2.76 mm to (177.7, 47.3), turned to -90 degrees
- moved C26 0.56 mm to (153.9, 81.7)
- moved R16 0.56 mm to (157.0, 81.8)
- moved C21 0.54 mm to (168.0, 81.6)
- moved R13 0.54 mm to (170.7, 81.6)
Routing:
- net GNDA: track 167.0 -> 176.8 mm
- net +3V3: track 158.9 -> 167.6 mm
- net GND: track 507.4 -> 513.7 mm
- net /IR_DEMOD: track 76.5 -> 79.3 mm, vias 1 -> 0
- net Net-(C22-Pad1): track 6.43 -> 8.95 mm
- net Net-(C23-Pad1): track 6.63 -> 5.90 mm
- net /LINEOUT_L: track 15.0 -> 15.6 mm
- net (no net): vias 4 -> 0
Other:
- board size 127.9 x 54.1 mm -> 127.9 x 53.5 mm
