File: pcb/ir-remote.kicad_sch (KiCad schematic)
At the start: 106 parts, among them J1 Conn_01x02, J12 Conn_01x04, J2 Conn_01x02, J3 Pins_02x04_P2.54mm_SMT, J4 USB-C_Receptacle_Molex_217179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, J5 Jack_RCA_Stereo, J6 Conn_01x03, J7 Jack_RCA_Stereo, J8 Conn_01x02, U1 STM32G431CBTx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

Commit message: SCH: saved in latest kicad (no changes)
Parts:
- removed R17, R18: 5.1k_0603, 4ms_Resistor:R_0603, symbol 4ms_Resistor_0603:5.1k_0603
- C40: value 10uF_0603_10V -> 2.2uF_0603_25V; symbol 4ms_Capacitor:10uF_0603_10V -> 4ms_Capacitor:2.2uF_0603_25V; Display 10uF/10V -> 2.2uF; JLCPCB ID C19702 -> C57895; Part Number GRM188R61A106KE69D -> GRM188R6YA225KA12D; Specifications 10uF, Min. 10V X5R 10% -> 2.2uF, Min 25V 10% X5R
- R2, R3, R6, R7, R8: value 33Ω_0603 -> 27Ω_0603; symbol 4ms_Resistor_0603:33Ω_0603 -> 4ms_Resistor_0603:27Ω_0603; Display 33Ω -> 27Ω; JLCPCB ID C23140 -> C137753; Part Number RC0603FR-0733RL -> RC0603FR-0727RL; Specifications 33Ω, 1%, 1/10W, 0603 -> 27Ω, 1%, 1/10W, 0603
Connections:
- no-connect marks 22 -> 24
Other:
- moved on the sheet: U6
